Commit message: improved tolerance for accurate ee pose

File: assets/meca500/meca.urdf (robot description, URDF)
Before this commit: robot meca_500_r3, 11 links, 10 joints
Links:
- removed link meca_gripper_finger1
- removed link meca_gripper_finger2
- removed link meca_gripper_link
Joints:
- removed joint meca_gripper_finger1_joint
- removed joint meca_gripper_finger2_joint
- removed joint meca_gripper_joint
