Commit message: end effector tool + collision checking

File: assets/tools/simple_tool.urdf (robot description, URDF)
Before this commit: robot simple_tool, 2 links, 1 joints
Links:
- link tool_base_link: geometry collision cylinder length=0.1 radius=0.03; visual cylinder length=0.1 radius=0.03
Joints:
- joint tool_base_to_tip: origin xyz=0 0 0.2 rpy=0 0 0 -> xyz=0 0 0.05 rpy=0 0 0
