Commit message: working code on linux, tested

File: assets/non_pii_face/non_pii_face_valid8.urdf (robot description, URDF)
Before this commit: robot non_pii_face_valid8, 1 links, 0 joints
Links:
- link face_link: geometry collision mesh filename=UR5-to-SuperClamp-withFoamForm.dae scale=0.0012 0.0012 0.0012; visual mesh filename=UR5-to-SuperClamp-withFoamForm.dae scale=0.0012 0.0012 0.0012

File: assets/tools/iphone.urdf (robot description, URDF)
Before this commit: robot iphone_tool, 2 links, 1 joints
Links:
- link tool_base_link: geometry collision box size=0.3 0.13 0.055; visual mesh filename=../tools/iphone.stl scale=0.04 0.04 0.04

File: assets/tools/optical_table.urdf (robot description, URDF)
Before this commit: robot optical_table, 1 links, 0 joints
Links:
- link table_link: geometry collision box size=2.1 1.1 1.04; visual mesh filename=optical_table.dae scale=1.4 1.37 1.17

File: assets/tx2_90xl/tx2_90xl_with_tx2_simple_tool.urdf (robot description, URDF)
Before this commit: robot staubli_tx2_90xl, 12 links, 11 joints
Links:
- removed link tx2_simple_tool_tool_base_link
- removed link tx2_simple_tool_tool_tip_link
- added link iphone::tool_base_link, mass 0.2; collision box size=0.3 0.13 0.055; visual mesh filename=../tools/iphone.stl scale=0.04 0.04 0.04
- added link iphone::tool_tip_link
Joints:
- removed joint tool_base_to_tip
- removed joint tx2_simple_tool_attach_joint
- added joint iphone::tool_base_to_tip: type fixed, parent iphone::tool_base_link, child iphone::tool_tip_link, origin xyz=0 0 0 rpy=0 0 0
- added joint iphone_attachment: type fixed, parent link_6, child iphone::tool_base_link, origin xyz=-0.08 0.0 0.03 rpy=0.0 0.0 0.0

File: assets/ur20/ur20_with_ur20_simple_tool.urdf (robot description, URDF)
Before this commit: robot ur20, 15 links, 14 joints
Links:
- removed link ur20_simple_tool_tool_base_link
- removed link ur20_simple_tool_tool_tip_link
- added link iphone::tool_base_link, mass 0.2; collision box size=0.3 0.13 0.055; visual mesh filename=../tools/iphone.stl scale=0.04 0.04 0.04
- added link iphone::tool_tip_link
Joints:
- removed joint tool_base_to_tip
- removed joint ur20_simple_tool_attach_joint
- added joint iphone::tool_base_to_tip: type fixed, parent iphone::tool_base_link, child iphone::tool_tip_link, origin xyz=0 0 0 rpy=0 0 0
- added joint iphone_attachment: type fixed, parent wrist_3_link, child iphone::tool_base_link, origin xyz=-0.08 0.0 0.03 rpy=0.0 0.0 0.0

File: assets/ur5e/ur5e_with_iphone_tool.urdf (robot description, URDF)
Before this commit: robot ur5e, 15 links, 14 joints
Links:
- removed link iphone_tool_tool_base_link
- removed link iphone_tool_tool_tip_link
- added link iphone::tool_base_link, mass 0.2; collision box size=0.3 0.13 0.055; visual mesh filename=../tools/iphone.stl scale=0.04 0.04 0.04
- added link iphone::tool_tip_link
Joints:
- removed joint iphone_tool_attach_joint
- removed joint tool_base_to_tip
- added joint iphone::tool_base_to_tip: type fixed, parent iphone::tool_base_link, child iphone::tool_tip_link, origin xyz=0 0 0 rpy=0 0 0
- added joint iphone_attachment: type fixed, parent wrist_3_link, child iphone::tool_base_link, origin xyz=-0.08 0.0 0.0 rpy=0.0 0.0 0.0
