Commit message: fix: smooth motion + mode switching for sim/real/both
Server:
- MoveIt ExecuteTrajectory action for proper trajectory execution
- Joint limits loaded (max_accel 5.0 rad/s², vel/accel scaling 0.1)
- robot_description_planning namespace wrapping for MoveIt
- Pre-flight robot readiness check (_ensure_robot_ready)
- New prepare_mode RPC for pre-execution validation
- All modes always reported as available (sim/real/both)
- Pre-flight validation in run_proto_sim for real/both modes

Client:
- All mode radio buttons always enabled (no graying out)
- Robot status indicator (green/amber/red dot)
- Pre-flight check dialog before real/both execution
  with Retry / Use Simulation / Cancel options

MoveIt config:
- move_group.launch.py rewritten with multi-path config loading
- joint_limits.yaml with acceleration limits (fixes TOTG default)
- Proper OMPL pipeline config format
- SRDF auto-generated by startup pipeline

Infra:
- Keepalive bash bug fix (|| echo 0 -> || true)
- Docker volume mounts for hot-reload of MoveIt config

File: valid8_cell_description/urdf/valid8_cell.urdf.xacro (robot description, xacro)
@@ -42,4 +42,32 @@
   <!-- Visual parameters -->
   <xacro:arg name="visual_parameters_file" default="$(find ur_description)/config/$(arg ur_type)/visual_parameters.yaml"/>
+  <!-- ========== ros2_control Parameters (required by UR driver) ========== -->
+  <xacro:arg name="robot_ip" default="0.0.0.0"/>
+  <xacro:arg name="use_fake_hardware" default="false"/>
+  <xacro:arg name="fake_sensor_commands" default="false"/>
+  <xacro:arg name="headless_mode" default="false"/>
+  <xacro:arg name="initial_positions_file" default="$(find ur_description)/config/initial_positions.yaml"/>
+  <xacro:arg name="script_filename" default=""/>
+  <xacro:arg name="output_recipe_filename" default=""/>
+  <xacro:arg name="input_recipe_filename" default=""/>
+  <xacro:arg name="reverse_ip" default="0.0.0.0"/>
+  <xacro:arg name="script_command_port" default="50004"/>
+  <xacro:arg name="reverse_port" default="50001"/>
+  <xacro:arg name="script_sender_port" default="50002"/>
+  <xacro:arg name="trajectory_port" default="50003"/>
+  <xacro:arg name="use_tool_communication" default="false"/>
+  <xacro:arg name="tool_voltage" default="0"/>
+  <xacro:arg name="tool_parity" default="0"/>
+  <xacro:arg name="tool_baud_rate" default="115200"/>
+  <xacro:arg name="tool_stop_bits" default="1"/>
+  <xacro:arg name="tool_rx_idle_chars" default="1.5"/>
+  <xacro:arg name="tool_tx_idle_chars" default="3.5"/>
+  <xacro:arg name="tool_device_name" default="/tmp/ttyUR"/>
+  <xacro:arg name="tool_tcp_port" default="54321"/>
+  <!-- Increase keep_alive_count significantly to give more time for commands -->
+  <!-- At 500Hz, count of 500 = 1000 seconds (~16 minutes) -->
+  <xacro:arg name="keep_alive_count" default="500"/>
+  <!-- Initial positions for simulation -->
+  <xacro:property name="initial_positions_file" value="$(arg initial_positions_file)"/>
   <!-- ========== World Link ========== -->
   <link name="world"/>
@@ -61,4 +89,27 @@
     physical_parameters_file="$(arg physical_parameters_file)"
     visual_parameters_file="$(arg visual_parameters_file)"
+    use_fake_hardware="$(arg use_fake_hardware)"
+    fake_sensor_commands="$(arg fake_sensor_commands)"
+    headless_mode="$(arg headless_mode)"
+    initial_positions="${xacro.load_yaml(initial_positions_file)}"
+    robot_ip="$(arg robot_ip)"
+    script_filename="$(arg script_filename)"
+    output_recipe_filename="$(arg output_recipe_filename)"
+    input_recipe_filename="$(arg input_recipe_filename)"
+    reverse_ip="$(arg reverse_ip)"
+    script_command_port="$(arg script_command_port)"
+    reverse_port="$(arg reverse_port)"
+    script_sender_port="$(arg script_sender_port)"
+    trajectory_port="$(arg trajectory_port)"
+    use_tool_communication="$(arg use_tool_communication)"
+    tool_voltage="$(arg tool_voltage)"
+    tool_parity="$(arg tool_parity)"
+    tool_baud_rate="$(arg tool_baud_rate)"
+    tool_stop_bits="$(arg tool_stop_bits)"
+    tool_rx_idle_chars="$(arg tool_rx_idle_chars)"
+    tool_tx_idle_chars="$(arg tool_tx_idle_chars)"
+    tool_device_name="$(arg tool_device_name)"
+    tool_tcp_port="$(arg tool_tcp_port)"
+    keep_alive_count="$(arg keep_alive_count)"
   >
     <!-- Robot base is directly on the mount (no additional offset) -->
