Commit message: fix: URDF visual rotations + increase tool collision depth
- Increase iPhone tool collision box depth: 0.055m → 0.08m
  (cuRobo spheres already cover this with radius=0.065)

- Rotate face_link visual +90° on X axis (rpy 0,0,-3.14 → 1.5708,0,-3.14)

- Rotate nakul_tool_base_link visual +90° on X axis (rpy 0,0,3.14 → 1.5708,0,3.14)

Applied to: both xacro copies (nvidia, server_new), reference URDF,
and cuRobo config comments.

File: assets/valid8_environment.urdf (robot description, URDF)
Before this commit: robot valid8_environment, 18 links, 17 joints
Links:
- link tool_base_link: geometry collision box size=0.3 0.13 0.08; visual mesh filename=package://simforge_server/assets/tools/iphone.stl scale=0.04 0.04 0.04

File: simforge_server_new/valid8_dual_cell_description/urdf/valid8_dual_cell_macro.xacro (robot description, xacro)
@@ -72,5 +72,5 @@
     <link name="face_link">
       <visual>
-        <origin xyz="0 -0.09 0" rpy="0 0 -3.14"/>
+        <origin xyz="0 -0.09 0" rpy="1.5708 0 -3.14"/>
         <geometry>
           <mesh filename="package://valid8_dual_cell_description/meshes/generix_human_head.stl" scale="0.001 0.001 0.001"/>
@@ -152,5 +152,5 @@
     <link name="nakul_tool_base_link">
       <visual>
-        <origin xyz="0 0 0" rpy="0 0 3.14"/>
+        <origin xyz="0 0 0" rpy="1.5708 0 3.14"/>
         <geometry>
           <mesh filename="package://valid8_dual_cell_description/meshes/iphone.stl" scale="0.04 0.04 0.04"/>
@@ -163,5 +163,5 @@
         <origin xyz="-0.065 0 0.02" rpy="1.5708 0 0"/>
         <geometry>
-          <box size="0.3 0.13 0.055"/>
+          <box size="0.3 0.13 0.08"/>
         </geometry>
       </collision>
