Commit message: cleanup: remove MoveIt references, dead code, and unused controllers
Summary of changes:

Deleted:
  - nodes/command_gateway_curobo_node.py.bak (2691-line monolith backup)

Removed dead code:
  - trajectory_executor._start_sim_trajectory() (defined, never called)
  - config.py: passthrough_controller, planning_group keys (unreferenced)
  - combined_controllers.yaml: 6 unused controller definitions
    (joint_trajectory_controller, forward_position_controller,
     passthrough_trajectory_controller for both robots)
  - valid8_dual_cell_description/package.xml: joint_state_publisher_gui dep

Cleaned MoveIt / old-architecture references from:
  - Dockerfile (removed 'Replaces MoveIt2 entirely', Jetson Thor refs)
  - docker-compose.yml (removed comparison comments)
  - start_server.sh (removed 'KEY DIFFERENCE from MoveIt version')
  - All 3 launch files (removed 'NOT launched: MoveIt2 move_group')
  - All 7 Python gateway modules (removed monolith/legacy/MoveIt noise)
  - Both package.xml files (updated descriptions, maintainer)
  - nakul_ur5e_curobo.yml (s/old MoveIt server/UR driver's/)

Renamed for clarity:
  - _run_legacy() → _run_pose_by_pose() in protocol_executor.py
  - 'Legacy fallback' → 'Pose-by-pose fallback' in comments/logs

Updated:
  - README.md: rewrote entirely — removed MoveIt comparison table,
    updated architecture diagram showing RTDE+ROS2 dual path,
    updated directory structure to reflect modular gateway
  - Dockerfile: added comment explaining why UR driver packages
    are still needed (sim uses ros2_control mock hardware)

File: simforge_server_nvidia/valid8_dual_cell_description/urdf/valid8_dual_cell_macro.xacro (robot description, xacro)
@@ -180,5 +180,5 @@
            maps tool_tip_link's frame so Y-axis aligns with the physical
            iPhone pointing direction. -->
-      <origin xyz="-0.08 0 0.05" rpy="1.57 0 0"/>
+      <origin xyz="-0.08 0 0.01" rpy="1.57 0 0"/>
       <parent link="nakul_wrist_3_link"/>
       <child link="nakul_tool_base_link"/>
