Commit message: SRDF-based self-collision ACM + collision-aware go-home
- Add scripts/generate_self_collision_ignore.py: converts MoveIt SRDF
  ACM (Allowed Collision Matrix) to cuRobo self_collision_ignore YAML.
  Uses MoveIt Setup Assistant's random-sampling collision analysis
  instead of manual guessing.

- Update nakul_ur5e_curobo.yml: SRDF-derived ACM — wrist_1↔tool_base
  and wrist_2↔tool_base are NO LONGER ignored (MoveIt confirms these
  CAN collide). Added shoulder↔forearm and upper_arm↔tool_base as safe
  to ignore. Set collision_sphere_buffer to 0.0.

- Update sahadev_ur5e_curobo.yml: SRDF-derived ACM — added non-adjacent
  safe pairs (shoulder↔forearm, forearm↔wrist_2/3, wrist_1↔wrist_3).

- Rewrite execute_home to use cuRobo plan_to_joints for collision-aware
  homing instead of raw RTDE moveJ. Falls back to moveJ only if cuRobo
  is unavailable. Prevents protective stops from tool-link collisions
  during go-home movements.

- Wire planner into TrajectoryExecutor via set_planner() so execute_home
  can access cuRobo planning.

- cuRobo planner: increase IK seeds to 100, planning attempts to 50,
  timeout to 30s, collision_activation_distance to 0.01.

- world_collision.yml: face cuboid 0.25→0.20 (matches URDF sphere r=0.1).

- ur20 tool URDF: fix collision origin Z sign.

File: assets/ur20/ur20_with_ur20_simple_tool.urdf (robot description, URDF)
Before this commit: robot ur20, 15 links, 14 joints
Links:
- link iphone::tool_base_link: geometry collision box size=0.3 0.13 0.06; visual mesh filename=../tools/iphone.stl scale=0.04 0.04 0.04
