Commit message: Fix new server to match old server's working behavior
Three critical changes to make the new server produce accurate robot poses:

1. URDF tool joint: Reverted to match old server's working values
   - xyz='-0.08 0 0.05' rpy='1.57 0 0' (was '0 0 0')
   - The 90° X rotation is required because the client's _look_at_quaternion
     generates Y-axis as the tool-forward direction
   - Collision box rpy also restored to '1.57 0 0'

2. Reference frame: Changed from 'world' to robot's base_link
   - get_environment_info now returns transforms relative to nakul_base_link
   - IK requests use nakul_base_link as frame_id (was 'world')
   - This matches the old server which uses 'base_link'
   - TF values are identical between old and new server

3. Workspace bounds: Added missing workspace parameters to planning
   - [-2,-2,-0.5] to [2,2,3] in robot's base_link frame
   - start_state.is_diff = False (explicit, matching old server)

File: simforge_server_new/valid8_dual_cell_description/urdf/valid8_dual_cell_macro.xacro (robot description, xacro)
@@ -161,5 +161,5 @@
       </visual>
       <collision>
-        <origin xyz="-0.065 0 0.02" rpy="0 0 0"/>
+        <origin xyz="-0.065 0 0.02" rpy="1.57 0 0"/>
         <geometry>
           <box size="0.3 0.13 0.055"/>
@@ -174,9 +174,11 @@
     <link name="nakul_tool_tip_link"/>
     <joint name="nakul_wrist_3_to_tool" type="fixed">
-      <!-- Tool attached to wrist_3_link matching Genesis convention:
-           xyz='-0.08 0 0' rpy='0 0 0' (no rotation).
-           This ensures tool_tip_link has the SAME orientation as wrist_3_link,
-           so IK + look-at (Z-axis pointing at target) works correctly. -->
-      <origin xyz="-0.08 0 0" rpy="0 0 0"/>
+      <!-- Tool attached to wrist_3_link with offset matching the old server:
+           xyz='-0.08 0 0.05' rpy='1.57 0 0' (90° X rotation).
+           The 90° X rotation is required because the client's _look_at_quaternion
+           generates Y-axis as the tool-forward direction, and this rotation
+           maps tool_tip_link's frame so Y-axis aligns with the physical
+           iPhone pointing direction. -->
+      <origin xyz="-0.08 0 0.05" rpy="1.57 0 0"/>
       <parent link="nakul_wrist_3_link"/>
       <child link="nakul_tool_base_link"/>

Commit message: fix: tool collision orientation + cuRobo sphere reorientation + servoJ safety
- Fix tool_base_link collision rpy in xacro: (0,0,0) -> (1.5708,0,0)
  to match reference valid8_environment.urdf. The 90-deg X rotation
  swaps the wide dimension (0.13m) from Y to Z, correctly representing
  the iPhone mount geometry.

- Reorient cuRobo tool collision spheres from Y-rows to Z-rows to
  match the corrected box orientation. Two rows at Z=+0.05 and Z=-0.01
  (was Y=+0.03 and Y=-0.03). Fixed sphere Y-center from 0.02 to 0.0.

- Add self_collision_buffer: 0.01 for nakul_tool_base_link to provide
  a small safety margin for tool-vs-robot-link collision checks.

- servoJ safety: replace recv-based isProtectiveStopped() check with
  isProgramRunning() + servoJ return value check. The recv interface
  silently fails during active servoJ streaming.

File: simforge_server_new/valid8_dual_cell_description/urdf/valid8_dual_cell_macro.xacro (robot description, xacro)
@@ -161,5 +161,5 @@
       </visual>
       <collision>
-        <origin xyz="-0.065 0 0.02" rpy="0 0 0"/>
+        <origin xyz="-0.065 0 0.02" rpy="1.5708 0 0"/>
         <geometry>
           <box size="0.3 0.13 0.055"/>

Commit message: cuRobo collision config overhaul: NVIDIA Lula spheres + home pose fix
- Replace hand-crafted collision spheres with NVIDIA's official
  Lula-generated spheres for all UR5e links (nakul + sahadev configs)
- Scale UR10e Lula spheres proportionally for UR20 (face_robot_ur20)
- Tool spheres: 3x5 grid at r=0.04 with self_collision_buffer=0.01
  (effective r=0.05 for self-collision, avoids home-pose false positives)
- collision_sphere_buffer: 0.005 (cuRobo default) for world collision
- Explicit self_collision_ignore matching official cuRobo UR5e config;
  wrist_2<->tool_base NOT ignored (fixes protective stop root cause)
- curobo_planner.py: merge hardcoded + computed self_collision_ignore
  (hardcoded pairs always preserved, computed pairs added on top)
- URDF tool collision box: 0.13 -> 0.16 in Y dimension (all xacros)
- face_robot_ur20 home_position aligned with sim initial_joint_positions
  (was [0,-pi/2,pi/2,-pi/2,-pi/2,0], now [0,-pi/2,0,-pi/2,0,0])
- Added mesh_link_names for all UR5e/UR20 links

File: simforge_server_new/valid8_dual_cell_description/urdf/valid8_dual_cell_macro.xacro (robot description, xacro)
@@ -163,5 +163,5 @@
         <origin xyz="-0.065 0 0.02" rpy="1.5708 0 0"/>
         <geometry>
-          <box size="0.3 0.13 0.08"/>
+          <box size="0.3 0.16 0.08"/>
         </geometry>
       </collision>

File: simforge_server_nvidia/environments/face_robot_ur20/description/urdf/face_robot_ur20_macro.xacro (robot description, xacro)
@@ -79,5 +79,5 @@
         <origin xyz="-0.065 0 0.02" rpy="1.5708 0 0"/>
         <geometry>
-          <box size="0.3 0.13 0.08"/>
+          <box size="0.3 0.16 0.08"/>
         </geometry>
       </collision>
